File: irradiance1.sch (KiCad schematic (older format))
At the start: 30 parts, among them J0 Conn_01x06, J4 CAN_In, J5 CAN_Out, J6 Battery, U1 ADM3055E, U2 Nucleo_L432KC, U7 CDSOT23-T24CAN

Commit message: Updated sheet details
Parts:
- J4, J5: symbol MPPT-rescue:CANConnector -> irradiance1-rescue:CANConnector-MPPT-rescue
- JP1: symbol MPPT-rescue:Jumper_NO_Small -> irradiance1-rescue:Jumper_NO_Small-MPPT-rescue
- R10, R25, R9: symbol MPPT-rescue:R -> irradiance1-rescue:R-MPPT-rescue
- U1: symbol MPPT-rescue:ADM3055E -> irradiance1-rescue:ADM3055E-MPPT-rescue
- U2: symbol Irradiance_board_parts:Nucleo_L432KC -> irradiance1-rescue:Nucleo_L432KC-Irradiance_board_parts
- U7: symbol MPPT-rescue:CDSOT23-T24CAN -> irradiance1-rescue:CDSOT23-T24CAN-MPPT-rescue
Changed lines of the file:
@@
 encoding utf-8
 Sheet 1 1
-Title ""
-Date ""
-Rev ""
-Comp ""
-Comment1 ""
-Comment2 ""
+Title "Standalone Irradiance Board"
+Date "2021-02-13"
+Rev "1.0"
+Comp "UTSVT"
+Comment1 "Matthew Yu"
+Comment2 "Jacob Pustilnik"
 Comment3 ""
 Comment4 ""
 $EndDescr
 $Comp
-L Irradiance_board_parts:Nucleo_L432KC U2
+L irradiance1-rescue:Nucleo_L432KC-Irradiance_board_parts U2
 U 1 1 5FAA17C6
 P 5500 2650
@@
 	4150 5100 4000 5100
 $Comp
-L MPPT-rescue:ADM3055E U1
+L irradiance1-rescue:ADM3055E-MPPT-rescue U1
 U 1 1 5FA7F796
 P 4850 5400
@@
 Connection ~ 7100 5150
 $Comp
-L MPPT-rescue:R R10
+L irradiance1-rescue:R-MPPT-rescue R10
 U 1 1 5FAC27E9
 P 8050 5450
@@
 $EndComp
 $Comp
-L MPPT-rescue:R R9
+L irradiance1-rescue:R-MPPT-rescue R9
 U 1 1 5FAC5664
 P 8250 5450
@@
 $EndComp
 $Comp
-L MPPT-rescue:CANConnector J4
+L irradiance1-rescue:CANConnector-MPPT-rescue J4
 U 1 1 5FACE509
 P 9300 5050
@@
 $EndComp
 $Comp
-L MPPT-rescue:CANConnector J5
+L irradiance1-rescue:CANConnector-MPPT-rescue J5
 U 1 1 5FACF8FF
 P 9300 5600
@@
 Connection ~ 7450 4900
 $Comp
-L MPPT-rescue:CDSOT23-T24CAN U7
+L irradiance1-rescue:CDSOT23-T24CAN-MPPT-rescue U7
 U 1 1 5FAD265B
 P 8250 4650
@@
 Connection ~ 7450 5150
 $Comp
-L MPPT-rescue:R R25
+L irradiance1-rescue:R-MPPT-rescue R25
 U 1 1 5FAD93D2
 P 5850 5950
@@
 NoConn ~ 5850 3000
 $Comp
-L MPPT-rescue:PWR_FLAG #FLG0101
+L irradiance1-rescue:PWR_FLAG-MPPT-rescue #FLG0101
 U 1 1 5FBE947A
 P 6350 2900
@@
 Connection ~ 8950 4900
 $Comp
-L MPPT-rescue:Jumper_NO_Small JP1
+L irradiance1-rescue:Jumper_NO_Small-MPPT-rescue JP1
 U 1 1 5FB266D0
 P 8150 5200
@@
 $EndComp
 $Comp
-L MPPT-rescue:+9VA #PWR0107
+L irradiance1-rescue:+9VA-MPPT-rescue #PWR0107
 U 1 1 5FDF1BB8
 P 5950 2800
@@
 	7050 4200 7250 4200
 $Comp
-L MPPT-rescue:+9VA #PWR0106
+L irradiance1-rescue:+9VA-MPPT-rescue #PWR0106
 U 1 1 5FDE8717
 P 7000 4000
